Commit message: Clean and organize Rovo ROS2 project

File: src/rovo_description/urdf/base.xacro (robot description, xacro)
@@ -1,29 +1,32 @@
 <?xml version="1.0"?>
 <robot xmlns:xacro="http://www.ros.org/wiki/xacro">
-<link name="base_link">
+  <link name="base_link">
+    <!-- ================= VISUAL ================= -->
     <visual>
-        <origin xyz="0 0 0.10"/>
-        <geometry>
-            <box size="0.60 0.45 0.20"/>
-        </geometry>
-        <material name="blue"/>
+      <origin xyz="0 0 0" rpy="0 0 0"/>
+      <geometry>
+        <box size="0.60 0.45 0.20"/>
+      </geometry>
+      <material name="blue"/>
     </visual>
+    <!-- ================= COLLISION ================= -->
     <collision>
-        <origin xyz="0 0 0.10"/>
-        <geometry>
-            <box size="0.60 0.45 0.20"/>
-        </geometry>
+      <origin xyz="0 0 0" rpy="0 0 0"/>
+      <geometry>
+        <box size="0.60 0.45 0.20"/>
+      </geometry>
     </collision>
+    <!-- ================= INERTIAL ================= -->
     <inertial>
-        <mass value="15"/>
-        <origin xyz="0 0 0.10"/>
-        <inertia
-            ixx="0.5"
-            iyy="0.5"
-            izz="0.5"
-            ixy="0"
-            ixz="0"
-            iyz="0"/>
+      <origin xyz="0 0 0" rpy="0 0 0"/>
+      <mass value="15"/>
+      <inertia
+        ixx="0.2656"
+        ixy="0"
+        ixz="0"
+        iyy="0.5750"
+        iyz="0"
+        izz="0.7813"/>
     </inertial>
-</link>
+  </link>
 </robot>

File: src/rovo_description/urdf/gazebo.xacro (robot description, xacro)
@@ -7,4 +7,6 @@
             filename="libgazebo_ros_joint_state_publisher.so">
       <update_rate>50</update_rate>
+      <joint_name>front_left_wheel_joint</joint_name>
+      <joint_name>front_right_wheel_joint</joint_name>
       <joint_name>left_wheel_joint</joint_name>
       <joint_name>right_wheel_joint</joint_name>
@@ -18,9 +20,9 @@
       </ros>
       <update_rate>50</update_rate>
-      <!-- Wheel joints -->
+      <!-- ONLY powered rear wheels -->
       <left_joint>left_wheel_joint</left_joint>
       <right_joint>right_wheel_joint</right_joint>
       <!-- Wheel dimensions -->
-      <wheel_separation>0.54</wheel_separation>
+      <wheel_separation>0.45</wheel_separation>
       <wheel_diameter>0.16</wheel_diameter>
       <!-- Motor limits -->
@@ -35,5 +37,21 @@
     </plugin>
   </gazebo>
-  <!-- Left Wheel Physics -->
+  <!-- Front Left Wheel -->
+  <gazebo reference="front_left_wheel">
+    <mu1>1.0</mu1>
+    <mu2>1.0</mu2>
+    <kp>1000000.0</kp>
+    <kd>100.0</kd>
+    <material>Gazebo/Black</material>
+  </gazebo>
+  <!-- Front Right Wheel -->
+  <gazebo reference="front_right_wheel">
+    <mu1>1.0</mu1>
+    <mu2>1.0</mu2>
+    <kp>1000000.0</kp>
+    <kd>100.0</kd>
+    <material>Gazebo/Black</material>
+  </gazebo>
+  <!-- Rear Left Wheel -->
   <gazebo reference="left_wheel">
     <mu1>1.0</mu1>
@@ -43,5 +61,5 @@
     <material>Gazebo/Black</material>
   </gazebo>
-  <!-- Right Wheel Physics -->
+  <!-- Rear Right Wheel -->
   <gazebo reference="right_wheel">
     <mu1>1.0</mu1>

File: src/rovo_description/urdf/sensors.xacro (robot description, xacro)
@@ -28,5 +28,5 @@
     <parent link="base_link"/>
     <child link="lidar_link"/>
-    <origin xyz="0.20 0 0.22"/>
+    <origin xyz="0 0 0.20"/>
   </joint>
   <!-- Camera -->

File: src/rovo_description/urdf/wheels.xacro (robot description, xacro)
@@ -1,65 +1,157 @@
 <?xml version="1.0"?>
 <robot xmlns:xacro="http://www.ros.org/wiki/xacro">
-<link name="left_wheel">
+  <!-- ================================================= -->
+  <!-- FRONT LEFT WHEEL -->
+  <!-- ================================================= -->
+  <link name="front_left_wheel">
     <visual>
-	<origin rpy="1.5708 0 0"/>
-        <geometry>
-            <cylinder radius="0.08" length="0.04"/>
-        </geometry>
-        <material name="black"/>
+      <origin xyz="0 0 0" rpy="1.5708 0 0"/>
+      <geometry>
+        <cylinder radius="0.08" length="0.04"/>
+      </geometry>
+      <material name="black"/>
     </visual>
     <collision>
-	<origin rpy="1.5708 0 0"/>
-        <geometry>
-            <cylinder radius="0.08" length="0.04"/>
-        </geometry>
+      <origin xyz="0 0 0" rpy="1.5708 0 0"/>
+      <geometry>
+        <cylinder radius="0.08" length="0.04"/>
+      </geometry>
     </collision>
     <inertial>
-        <mass value="1"/>
-        <inertia
-            ixx="0.001"
-            ixy="0"
-            ixz="0"
-            iyy="0.001"
-            iyz="0"
-            izz="0.001"/>
+      <origin xyz="0 0 0"/>
+      <mass value="0.5"/>
+      <inertia
+        ixx="0.0017"
+        ixy="0"
+        ixz="0"
+        iyy="0.0008"
+        iyz="0"
+        izz="0.0017"/>
     </inertial>
-</link>
-<link name="right_wheel">
+  </link>
+  <!-- ================================================= -->
+  <!-- FRONT RIGHT WHEEL -->
+  <!-- ================================================= -->
+  <link name="front_right_wheel">
     <visual>
-	<origin rpy="1.5708 0 0"/>
-        <geometry>
-            <cylinder radius="0.08" length="0.04"/>
-        </geometry>
-        <material name="black"/>
+      <origin xyz="0 0 0" rpy="1.5708 0 0"/>
+      <geometry>
+        <cylinder radius="0.08" length="0.04"/>
+      </geometry>
+      <material name="black"/>
     </visual>
     <collision>
-	<origin rpy="1.5708 0 0"/>
-        <geometry>
-            <cylinder radius="0.08" length="0.04"/>
-        </geometry>
+      <origin xyz="0 0 0" rpy="1.5708 0 0"/>
+      <geometry>
+        <cylinder radius="0.08" length="0.04"/>
+      </geometry>
     </collision>
     <inertial>
-        <mass value="1"/>
-        <inertia
-            ixx="0.001"
-            ixy="0"
-            ixz="0"
-            iyy="0.001"
-            iyz="0"
-            izz="0.001"/>
+      <origin xyz="0 0 0"/>
+      <mass value="0.5"/>
+      <inertia
+        ixx="0.0017"
+        ixy="0"
+        ixz="0"
+        iyy="0.0008"
+        iyz="0"
+        izz="0.0017"/>
     </inertial>
-</link>
-<joint name="left_wheel_joint" type="continuous">
+  </link>
+  <!-- ================================================= -->
+  <!-- REAR LEFT WHEEL -->
+  <!-- This is a powered drive wheel -->
+  <!-- ================================================= -->
+  <link name="left_wheel">
+    <visual>
+      <origin xyz="0 0 0" rpy="1.5708 0 0"/>
+      <geometry>
+        <cylinder radius="0.08" length="0.04"/>
+      </geometry>
+      <material name="black"/>
+    </visual>
+    <collision>
+      <origin xyz="0 0 0" rpy="1.5708 0 0"/>
+      <geometry>
+        <cylinder radius="0.08" length="0.04"/>
+      </geometry>
+    </collision>
+    <inertial>
+      <origin xyz="0 0 0"/>
+      <mass value="1.0"/>
+      <inertia
+        ixx="0.0034"
+        ixy="0"
+        ixz="0"
+        iyy="0.0016"
+        iyz="0"
+        izz="0.0034"/>
+    </inertial>
+  </link>
+  <!-- ================================================= -->
+  <!-- REAR RIGHT WHEEL -->
+  <!-- This is a powered drive wheel -->
+  <!-- ================================================= -->
+  <link name="right_wheel">
+    <visual>
+      <origin xyz="0 0 0" rpy="1.5708 0 0"/>
+      <geometry>
+        <cylinder radius="0.08" length="0.04"/>
+      </geometry>
+      <material name="black"/>
+    </visual>
+    <collision>
+      <origin xyz="0 0 0" rpy="1.5708 0 0"/>
+      <geometry>
+        <cylinder radius="0.08" length="0.04"/>
+      </geometry>
+    </collision>
+    <inertial>
+      <origin xyz="0 0 0"/>
+      <mass value="1.0"/>
+      <inertia
+        ixx="0.0034"
+        ixy="0"
+        ixz="0"
+        iyy="0.0016"
+        iyz="0"
+        izz="0.0034"/>
+    </inertial>
+  </link>
+  <!-- ================================================= -->
+  <!-- FRONT LEFT WHEEL JOINT -->
+  <!-- ================================================= -->
+  <joint name="front_left_wheel_joint" type="continuous">
+    <parent link="base_link"/>
+    <child link="front_left_wheel"/>
+    <origin xyz="0.20 0.225 -0.10" rpy="0 0 0"/>
+    <axis xyz="0 1 0"/>
+  </joint>
+  <!-- ================================================= -->
+  <!-- FRONT RIGHT WHEEL JOINT -->
+  <!-- ================================================= -->
+  <joint name="front_right_wheel_joint" type="continuous">
+    <parent link="base_link"/>
+    <child link="front_right_wheel"/>
+    <origin xyz="0.20 -0.225 -0.10" rpy="0 0 0"/>
+    <axis xyz="0 1 0"/>
+  </joint>
+  <!-- ================================================= -->
+  <!-- REAR LEFT DRIVE WHEEL JOINT -->
+  <!-- ================================================= -->
+  <joint name="left_wheel_joint" type="continuous">
     <parent link="base_link"/>
     <child link="left_wheel"/>
-    <origin xyz="0 0.27 0.08"/>
+    <origin xyz="-0.20 0.225 -0.10" rpy="0 0 0"/>
     <axis xyz="0 1 0"/>
-</joint>
-<joint name="right_wheel_joint" type="continuous">
+  </joint>
+  <!-- ================================================= -->
+  <!-- REAR RIGHT DRIVE WHEEL JOINT -->
+  <!-- ================================================= -->
+  <joint name="right_wheel_joint" type="continuous">
     <parent link="base_link"/>
     <child link="right_wheel"/>
-    <origin xyz="0 -0.27 0.08"/>
+    <origin xyz="-0.20 -0.225 -0.10" rpy="0 0 0"/>
     <axis xyz="0 1 0"/>
-</joint>
+  </joint>
 </robot>
